File: PCB/MainBoard/MainBoard.kicad_pcb (KiCad board)
At the start: 2 copper layers, 177.8 x 120.7 mm, 136 parts, among them J1 Fan, J2 PowerIn, J3 AuxPowerIn, J4 LCD Display, J5 SWD, J6 FrontPanel, J7 PowerOut, K1 OUT_A_ENABLE_RELAY, K2 OUT_B_ENABLE_RELAY, K3 Relay_SPDT_Panasonic_ALQ105, K4 Relay_SPDT_Panasonic_ALQ105, K5 Relay_SPDT_Panasonic_ALQ105, M1 Fan, Q1 TIP41C, Q10 2N2222, Q11 TIP41C, Q12 TIP41C, Q2 TSM2302CX, Q3 TIP41C, Q4 TSM2302CX, Q5 TSM2302CX, Q6 TSM2302CX, Q7 TSM2302CX, Q8 TSM2302CX, Q9 2N2222, U1 LTC2631CTS8-HZ12, U10 LM35-NEB, U2 LTC2631CTS8-HZ12, U3 MCP3428, U4 2SC5200NS1_E_S, U5 LT1490CN8PBF, U6 2SC5200NS1_E_S, U7 STM32F411RETx, U8 MCP1703A-3302_SOT223, U9 LM35-NEB, Y1 24MHz, Y2 32k768

Commit message: Fix minor issues in PCB
Fixed decoupling capacitors connectivbity
Added test points to several networks
Parts:
- added TP1: TP_CH_A_MAINPWR_CTRL, TestPoint:TestPoint_THTPad_D2.0mm_Drill1.0mm, F.Cu at (409.1, 102.3)
- added TP10: TP_CH_B_MAINPWR_CTRL, TestPoint:TestPoint_THTPad_D2.0mm_Drill1.0mm, F.Cu at (409.1, 189.0)
- added TP13: OPAMP_CH_B_INV, TestPoint:TestPoint_THTPad_D2.0mm_Drill1.0mm, F.Cu at (284.3, 106.8)
- added TP3: TP_DAC_VOUT_CH_A, TestPoint:TestPoint_THTPad_D2.0mm_Drill1.0mm, F.Cu at (263.1, 109.9)
- added TP5: TP_DAC_VOUT_CH_B, TestPoint:TestPoint_THTPad_D2.0mm_Drill1.0mm, F.Cu at (281.0, 106.8)
- added TP8: OPAMP_CH_A_INV, TestPoint:TestPoint_THTPad_D2.0mm_Drill1.0mm, F.Cu at (263.1, 106.1)
- moved C9 6.31 mm to (278.0, 115.2), turned to 180 degrees
- moved C8 6.25 mm to (268.5, 109.1), turned to 0 degrees
- moved C6 5.20 mm to (267.6, 111.2), turned to 0 degrees
- moved U2 4.21 mm to (278.5, 110.3), turned to 180 degrees
- moved C7 3.85 mm to (278.8, 113.1), turned to 180 degrees
- turned C17 to 180 degrees
- renumbered TP6 to TP11, TP7 to TP12, TP8 to TP14, TP9 to TP15, TP10 to TP16, TP1 to TP2, TP2 to TP4, TP3 to TP6, TP4 to TP7, TP5 to TP9
Connections:
- net Net-(R16-Pad1) renamed /CH_A_INV
- net Net-(R20-Pad1) renamed /CH_B_INV
- net Net-(U1-Pad7) renamed /DAC_VOUT_CH_A
- net Net-(U2-Pad7) renamed /DAC_VOUT_CH_B
Routing:
- net +5V: track 611.8 -> 546.5 mm, vias 16 -> 14
- net Net-(C11-Pad2): track 42.4 -> 58.7 mm
- net GND: track 39.3 -> 53.4 mm
- net Net-(C4-Pad2): track 57.1 -> 68.8 mm
- net +3V3: track 133.2 -> 127.9 mm
- net I2C1_SDA: track 126.9 -> 121.9 mm, vias 0 -> 2
- net /CH_A_INV: track 13.3 -> 18.3 mm
- net /DAC_VOUT_CH_A: track 13.8 -> 18.5 mm
- net /DAC_VOUT_CH_B: track 13.3 -> 9.31 mm, vias 2 -> 0
- net /CH_B_INV: track 13.8 -> 17.0 mm
- net I2C1_SCL: track 117.9 -> 116.9 mm
